File: efr32mg21_devboard/efr32mg21_devboard.kicad_pcb (KiCad board)
At the start: 2 copper layers, 19 parts, among them CON1 CORTEX-DEBUGGER, U1 EFR32MG21A020F768IM32-BR, Y1 38.4MHz, Y2 32.768k

Commit message: pcb
Parts:
- added J1: Conn_01x10, Connector_PinHeader_2.54mm:PinHeader_1x10_P2.54mm_Vertical, F.Cu at (163.9, 89.1)
- added J2: microusb, mybays_connector:MICRO-USB_MICRO-USB-17, F.Cu at (150.4, 115.8)
- added J3: Conn_01x10, Connector_PinHeader_2.54mm:PinHeader_1x10_P2.54mm_Vertical, F.Cu at (128.8, 87.3)
- added U2: TLV70033_SOT23-5, Package_TO_SOT_SMD:SOT-23-5, F.Cu at (140.1, 110.7)
Other:
- board outline added: 50 x 50 mm

Commit message: pcb
Parts:
- moved J3 1.05 mm to (129.8, 87.8)
Connections:
- J1 pad 10: Net-(J1-Pad10) -> PD04
- J1 pad 2: Net-(J1-Pad2) -> PC05
- J1 pad 3: Net-(J1-Pad3) -> PC04
- J1 pad 4: Net-(J1-Pad4) -> PC03
- J1 pad 5: Net-(J1-Pad5) -> PC02
- J1 pad 6: Net-(J1-Pad6) -> PC01
- J1 pad 7: Net-(J1-Pad7) -> PC00
- J1 pad 8: Net-(J1-Pad8) -> PD02
- J1 pad 9: Net-(J1-Pad9) -> PD03
- J3 pad 1: Net-(J3-Pad1) -> PB01
- J3 pad 2: Net-(J3-Pad2) -> PB00
- J3 pad 3: Net-(J3-Pad3) -> PA00
- J3 pad 4: Net-(J3-Pad4) -> PA01
- J3 pad 5: Net-(J3-Pad5) -> PA02
- J3 pad 6: Net-(J3-Pad6) -> PA03
- J3 pad 7: Net-(J3-Pad7) -> PA04
- J3 pad 8: Net-(J3-Pad8) -> PA05
- J3 pad 9: Net-(J3-Pad9) -> PA06
Changed lines of the file:
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@@
     (zones 0)
     (modules 23)
-    (nets 66)
+    (nets 48)
   )
   (page A4)
@@
   (net 33 "Net-(CON1-Pad4)")
   (net 34 "Net-(CON1-Pad1)")
-  (net 35 "Net-(J1-Pad10)")
-  (net 36 "Net-(J1-Pad9)")
-  (net 37 "Net-(J1-Pad8)")
-  (net 38 "Net-(J1-Pad7)")
-  (net 39 "Net-(J1-Pad6)")
-  (net 40 "Net-(J1-Pad5)")
-  (net 41 "Net-(J1-Pad4)")
-  (net 42 "Net-(J1-Pad3)")
-  (net 43 "Net-(J1-Pad2)")
-  (net 44 "Net-(J1-Pad1)")
-  (net 45 "Net-(J2-Pad0)")
-  (net 46 "Net-(J2-Pad1)")
-  (net 47 "Net-(J2-Pad2)")
-  (net 48 "Net-(J2-Pad3)")
-  (net 49 "Net-(J2-Pad4)")
-  (net 50 "Net-(J2-Pad5)")
-  (net 51 "Net-(U2-Pad5)")
-  (net 52 "Net-(U2-Pad4)")
-  (net 53 "Net-(U2-Pad3)")
-  (net 54 "Net-(U2-Pad2)")
-  (net 55 "Net-(U2-Pad1)")
-  (net 56 "Net-(J3-Pad10)")
-  (net 57 "Net-(J3-Pad9)")
-  (net 58 "Net-(J3-Pad8)")
-  (net 59 "Net-(J3-Pad7)")
-  (net 60 "Net-(J3-Pad6)")
-  (net 61 "Net-(J3-Pad5)")
-  (net 62 "Net-(J3-Pad4)")
-  (net 63 "Net-(J3-Pad3)")
-  (net 64 "Net-(J3-Pad2)")
-  (net 65 "Net-(J3-Pad1)")
+  (net 35 "Net-(J1-Pad1)")
+  (net 36 "Net-(J2-Pad0)")
+  (net 37 "Net-(J2-Pad1)")
+  (net 38 "Net-(J2-Pad2)")
+  (net 39 "Net-(J2-Pad3)")
+  (net 40 "Net-(J2-Pad4)")
+  (net 41 "Net-(J2-Pad5)")
+  (net 42 "Net-(U2-Pad5)")
+  (net 43 "Net-(U2-Pad4)")
+  (net 44 "Net-(U2-Pad3)")
+  (net 45 "Net-(U2-Pad2)")
+  (net 46 "Net-(U2-Pad1)")
+  (net 47 "Net-(J3-Pad10)")
   (net_class Default "This is the default net class."
     (clearance 0.2)
@@
     (add_net "Net-(CON1-Pad8)")
     (add_net "Net-(J1-Pad1)")
-    (add_net "Net-(J1-Pad10)")
-    (add_net "Net-(J1-Pad2)")
-    (add_net "Net-(J1-Pad3)")
-    (add_net "Net-(J1-Pad4)")
-    (add_net "Net-(J1-Pad5)")
-    (add_net "Net-(J1-Pad6)")
-    (add_net "Net-(J1-Pad7)")
-    (add_net "Net-(J1-Pad8)")
-    (add_net "Net-(J1-Pad9)")
     (add_net "Net-(J2-Pad0)")
     (add_net "Net-(J2-Pad1)")
@@
     (add_net "Net-(J2-Pad4)")
     (add_net "Net-(J2-Pad5)")
-    (add_net "Net-(J3-Pad1)")
     (add_net "Net-(J3-Pad10)")
-    (add_net "Net-(J3-Pad2)")
-    (add_net "Net-(J3-Pad3)")
-    (add_net "Net-(J3-Pad4)")
-    (add_net "Net-(J3-Pad5)")
-    (add_net "Net-(J3-Pad6)")
-    (add_net "Net-(J3-Pad7)")
-    (add_net "Net-(J3-Pad8)")
-    (add_net "Net-(J3-Pad9)")
     (add_net "Net-(U1-Pad31)")
     (add_net "Net-(U1-Pad32)")
@@
   )
   (module Connector_PinHeader_2.54mm:PinHeader_1x10_P2.54mm_Vertical (layer F.Cu)
-    (at 128.82626 87.31758)
+    (at 129.76098 87.7951)
     (descr "Through hole straight pin header, 1x10, 2.54mm pitch, single row")
     (tags "Through hole pin header THT 1x10 2.54mm single row")
@@
     (fp_line (start 1.8 -1.8) (end -1.8 -1.8) (layer F.CrtYd) (width 0.05))
     (pad 10 thru_hole oval (at 0 22.86) (size 1.7 1.7) (drill 1) (layers *.Cu *.Mask)
-      (net 56 "Net-(J3-Pad10)"))
+      (net 47 "Net-(J3-Pad10)"))
     (pad 9 thru_hole oval (at 0 20.32) (size 1.7 1.7) (drill 1) (layers *.Cu *.Mask)
-      (net 57 "Net-(J3-Pad9)"))
+      (net 15 PA06))
     (pad 8 thru_hole oval (at 0 17.78) (size 1.7 1.7) (drill 1) (layers *.Cu *.Mask)
-      (net 58 "Net-(J3-Pad8)"))
+      (net 16 PA05))
     (pad 7 thru_hole oval (at 0 15.24) (size 1.7 1.7) (drill 1) (layers *.Cu *.Mask)
-      (net 59 "Net-(J3-Pad7)"))
+      (net 17 PA04))
     (pad 6 thru_hole oval (at 0 12.7) (size 1.7 1.7) (drill 1) (layers *.Cu *.Mask)
-      (net 60 "Net-(J3-Pad6)"))
+      (net 18 PA03))
     (pad 5 thru_hole oval (at 0 10.16) (size 1.7 1.7) (drill 1) (layers *.Cu *.Mask)
-      (net 61 "Net-(J3-Pad5)"))
+      (net 19 PA02))
     (pad 4 thru_hole oval (at 0 7.62) (size 1.7 1.7) (drill 1) (layers *.Cu *.Mask)
-      (net 62 "Net-(J3-Pad4)"))
+      (net 20 PA01))
     (pad 3 thru_hole oval (at 0 5.08) (size 1.7 1.7) (drill 1) (layers *.Cu *.Mask)
-      (net 63 "Net-(J3-Pad3)"))
+      (net 21 PA00))
     (pad 2 thru_hole oval (at 0 2.54) (size 1.7 1.7) (drill 1) (layers *.Cu *.Mask)
-      (net 64 "Net-(J3-Pad2)"))
+      (net 22 PB00))
     (pad 1 thru_hole rect (at 0 0) (size 1.7 1.7) (drill 1) (layers *.Cu *.Mask)
-      (net 65 "Net-(J3-Pad1)"))
+      (net 23 PB01))
     (model ${KISYS3DMOD}/Connector_PinHeader_2.54mm.3dshapes/PinHeader_1x10_P2.54mm_Vertical.wrl
       (at (xyz 0 0 0))
@@
     (fp_line (start 0.9 -1.55) (end 0.9 1.55) (layer F.Fab) (width 0.1))
     (pad 5 smd rect (at 1.1 -0.95) (size 1.06 0.65) (layers F.Cu F.Paste F.Mask)
-      (net 51 "Net-(U2-Pad5)"))
+      (net 42 "Net-(U2-Pad5)"))
     (pad 4 smd rect (at 1.1 0.95) (size 1.06 0.65) (layers F.Cu F.Paste F.Mask)
-      (net 52 "Net-(U2-Pad4)"))
+      (net 43 "Net-(U2-Pad4)"))
     (pad 3 smd rect (at -1.1 0.95) (size 1.06 0.65) (layers F.Cu F.Paste F.Mask)
-      (net 53 "Net-(U2-Pad3)"))
+      (net 44 "Net-(U2-Pad3)"))
     (pad 2 smd rect (at -1.1 0) (size 1.06 0.65) (layers F.Cu F.Paste F.Mask)
-      (net 54 "Net-(U2-Pad2)"))
+      (net 45 "Net-(U2-Pad2)"))
     (pad 1 smd rect (at -1.1 -0.95) (size 1.06 0.65) (layers F.Cu F.Paste F.Mask)
-      (net 55 "Net-(U2-Pad1)"))
+      (net 46 "Net-(U2-Pad1)"))
     (model ${KISYS3DMOD}/Package_TO_SOT_SMD.3dshapes/SOT-23-5.wrl
       (at (xyz 0 0 0))
@@
     (fp_line (start 3.685032 -0.679323) (end 3.685032 0.149225) (layer F.SilkS) (width 0.254))
     (pad 0 smd rect (at 3.24993 1.080516 180) (size 1.499997 1.400048) (layers F.Cu F.Paste F.Mask)
-      (net 45 "Net-(J2-Pad0)"))
+      (net 36 "Net-(J2-Pad0)"))
     (pad 0 smd rect (at -3.24993 1.080516 180) (size 1.499997 1.400048) (layers F.Cu F.Paste F.Mask)
-      (net 45 "Net-(J2-Pad0)"))
+      (net 36 "Net-(J2-Pad0)"))
     (pad 0 smd rect (at 3.074922 -1.660398) (size 2.5 1.499997) (layers F.Cu F.Paste F.Mask)
-      (net 45 "Net-(J2-Pad0)"))
+      (net 36 "Net-(J2-Pad0)"))
     (pad 0 smd rect (at -3.074922 -1.660398 90) (size 1.499997 2.5) (layers F.Cu F.Paste F.Mask)
-      (net 45 "Net-(J2-Pad0)"))
+      (net 36 "Net-(J2-Pad0)"))
     (pad 1 smd rect (at 1.296416 1.660652 270) (size 1.799996 0.399999) (layers F.Cu F.Paste F.Mask)
-      (net 46 "Net-(J2-Pad1)"))
+      (net 37 "Net-(J2-Pad1)"))
     (pad 2 smd rect (at 0.646176 1.660652 270) (size 1.799996 0.399999) (layers F.Cu F.Paste F.Mask)
-      (net 47 "Net-(J2-Pad2)"))
+      (net 38 "Net-(J2-Pad2)"))
     (pad 3 smd rect (at -0.004064 1.660652 270) (size 1.799996 0.399999) (layers F.Cu F.Paste F.Mask)
-      (net 48 "Net-(J2-Pad3)"))
+      (net 39 "Net-(J2-Pad3)"))
     (pad 4 smd rect (at -0.654304 1.660652 270) (size 1.799996 0.399999) (layers F.Cu F.Paste F.Mask)
-      (net 49 "Net-(J2-Pad4)"))
+      (net 40 "Net-(J2-Pad4)"))
     (pad 5 smd rect (at -1.304544 1.660652 270) (size 1.799996 0.399999) (layers F.Cu F.Paste F.Mask)
-      (net 50 "Net-(J2-Pad5)"))
+      (net 41 "Net-(J2-Pad5)"))
     (pad "" np_thru_hole circle (at 1.9939 0.999236 180) (size 0.700024 0.700024) (drill 0.700024) (layers *.Cu *.Mask))
     (pad "" np_thru_hole circle (at -2.00406 0.999236 180) (size 0.700024 0.700024) (drill 0.700024) (layers *.Cu *.Mask))
@@
     (fp_line (start 1.8 -1.8) (end -1.8 -1.8) (layer F.CrtYd) (width 0.05))
     (pad 10 thru_hole oval (at 0 22.86) (size 1.7 1.7) (drill 1) (layers *.Cu *.Mask)
-      (net 35 "Net-(J1-Pad10)"))
+      (net 14 PD04))
     (pad 9 thru_hole oval (at 0 20.32) (size 1.7 1.7) (drill 1) (layers *.Cu *.Mask)
-      (net 36 "Net-(J1-Pad9)"))
+      (net 13 PD03))
     (pad 8 thru_hole oval (at 0 17.78) (size 1.7 1.7) (drill 1) (layers *.Cu *.Mask)
-      (net 37 "Net-(J1-Pad8)"))
+      (net 12 PD02))
     (pad 7 thru_hole oval (at 0 15.24) (size 1.7 1.7) (drill 1) (layers *.Cu *.Mask)
-      (net 38 "Net-(J1-Pad7)"))
+      (net 30 PC00))
     (pad 6 thru_hole oval (at 0 12.7) (size 1.7 1.7) (drill 1) (layers *.Cu *.Mask)
-      (net 39 "Net-(J1-Pad6)"))
+      (net 29 PC01))
     (pad 5 thru_hole oval (at 0 10.16) (size 1.7 1.7) (drill 1) (layers *.Cu *.Mask)
-      (net 40 "Net-(J1-Pad5)"))
+      (net 28 PC02))
     (pad 4 thru_hole oval (at 0 7.62) (size 1.7 1.7) (drill 1) (layers *.Cu *.Mask)
-      (net 41 "Net-(J1-Pad4)"))
+      (net 27 PC03))
     (pad 3 thru_hole oval (at 0 5.08) (size 1.7 1.7) (drill 1) (layers *.Cu *.Mask)
-      (net 42 "Net-(J1-Pad3)"))
+      (net 26 PC04))
     (pad 2 thru_hole oval (at 0 2.54) (size 1.7 1.7) (drill 1) (layers *.Cu *.Mask)
-      (net 43 "Net-(J1-Pad2)"))
+      (net 25 PC05))
     (pad 1 thru_hole rect (at 0 0) (size 1.7 1.7) (drill 1) (layers *.Cu *.Mask)
-      (net 44 "Net-(J1-Pad1)"))
+      (net 35 "Net-(J1-Pad1)"))
     (model ${KISYS3DMOD}/Connector_PinHeader_2.54mm.3dshapes/PinHeader_1x10_P2.54mm_Vertical.wrl
       (at (xyz 0 0 0))

Commit message: v1.0
Parts:
- added C8: C, Capacitor_SMD:C_1206_3216Metric, F.Cu at (142.5, 116.4)
- added C9: C, Capacitor_SMD:C_1206_3216Metric, F.Cu at (156.3, 116.7)
- added J4: Conn_02x02_Counter_Clockwise, Connector_PinHeader_2.54mm:PinHeader_2x02_P2.54mm_Vertical, F.Cu at (136.0, 115.0)
- added J5: Conn_02x02_Counter_Clockwise, Connector_PinHeader_2.54mm:PinHeader_2x02_P2.54mm_Vertical, F.Cu at (160.0, 115.0)
- moved U2 14.6 mm to (154.7, 111.5)
- moved CON1 13.3 mm to (142.4, 109.9), turned to 270 degrees
- moved C100 3.65 mm to (157.1, 92.0)
- moved C101 3.65 mm to (156.1, 92.0)
- moved L100 3.65 mm to (158.3, 91.4)
- moved Y1 3.56 mm to (157.3, 95.3)
- moved J1 3.33 mm to (167.0, 88.0)
- moved J3 3.25 mm to (133.0, 88.0)
- moved Y2 3.10 mm to (156.8, 103.5), turned to 180 degrees
- moved L2 1.95 mm to (154.0, 82.0)
- moved J2 1.35 mm to (149.2, 116.4)
Connections:
- CON1 pad 10: Net-(CON1-Pad10) -> PB00
- CON1 pad 8: Net-(CON1-Pad8) -> PB01
- J1 pad 1: Net-(J1-Pad1) -> GND
- J2 pad 0: Net-(J2-Pad0) -> GND
- J2 pad 1: Net-(J2-Pad1) -> Net-(C8-Pad1)
- J2 pad 5: Net-(J2-Pad5) -> GND
- J3 pad 10: Net-(J3-Pad10) -> GND
- U2 pad 1: Net-(U2-Pad1) -> Net-(C8-Pad1)
- U2 pad 2: Net-(U2-Pad2) -> GND
- U2 pad 3: Net-(U2-Pad3) -> Net-(C8-Pad1)
- U2 pad 5: Net-(U2-Pad5) -> +3V3
Routing:
- net GND: track 21.4 -> 189.7 mm, vias 0 -> 19
- net +3V3: track 11.0 -> 85.2 mm, vias 0 -> 3
- net PB01: track 0.00 -> 55.9 mm
- net PB00: track 0.00 -> 49.4 mm
- net PA01: track 0.00 -> 33.4 mm
- net PA02: track 0.00 -> 27.9 mm, vias 0 -> 1
- net PD04: track 0.00 -> 21.6 mm
- net PA06: track 0.00 -> 20.1 mm
- net PD03: track 0.00 -> 20.0 mm
- net PC05: track 0.00 -> 18.7 mm
- net PD02: track 0.00 -> 18.5 mm
- net RESETn: track 0.00 -> 18.4 mm, vias 0 -> 1
- net PA05: track 0.00 -> 18.2 mm
- net PC04: track 0.00 -> 17.8 mm
- net Net-(C8-Pad1): track 0.00 -> 17.4 mm
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- added copper zone on B.Cu, net (none)
- added copper zone on F.Cu, net GND
Other:
- board size 50 x 50 mm -> 40 x 40 mm
- board text added: "3V3"
- board text added: "GND"
- board text added: "PA00"
- board text added: "PA01"
- board text added: "PA02"
- board text added: "PA03"
- board text added: "PA04"
- board text added: "PA05"
- board text added: "PA06"
- board text added: "PB00"
- board text added: "PB01"
- board text added: "PC00"
- board text added: "PC01"
- board text added: "PC02"
- board text added: "PC03"
- board text added: "PC04"
- board text added: "PC05"
- board text added: "PD02"
- board text added: "PD03"
- board text added: "PD04"
